File: kicad/kicad.kicad_pcb (KiCad board)
At the start: 2 copper layers, 340.6 x 156.5 mm, 211 parts, among them SW1 SW_Push, SW10 SW_Push, SW11 SW_Push, SW12 SW_Push, SW13 SW_Push, SW14 SW_Push, SW15 SW_Push, SW16 SW_Push, SW17 SW_Push, SW18 SW_Push, SW19 SW_Push, SW2 SW_Push, SW20 SW_Push, SW21 SW_Push, SW22 SW_Push, SW23 SW_Push, SW24 SW_Push, SW25 SW_Push, SW26 SW_Push, SW27 SW_Push, SW28 SW_Push, SW29 SW_Push, SW3 SW_Push, SW30 SW_Push, SW31 SW_Push, SW32 SW_Push, SW33 SW_Push, SW34 SW_Push, SW35 SW_Push, SW36 SW_Push, SW37 SW_Push, SW38 SW_Push, SW39 SW_Push, SW4 SW_Push, SW40 SW_Push, SW41 SW_Push, SW42 SW_Push, SW43 SW_Push, SW44 SW_Push, SW45 SW_Push, SW46 SW_Push, SW47 SW_Push, SW48 SW_Push, SW49 SW_Push, SW5 SW_Push, SW50 SW_Push, SW51 SW_Push, SW52 SW_Push, SW53 SW_Push, SW54 SW_Push, SW55 SW_Push, SW56 SW_Push, SW57 SW_Push, SW58 SW_Push, SW59 SW_Push, SW6 SW_Push, SW60 SW_Push, SW61 SW_Push, SW7 SW_Push, SW8 SW_Push, SW9 SW_Push

Commit message: Reattempt to match forge requirments: rmved sm useless vias and added in other places
Routing:
- net Net-(RGB15-DOUT): track 346.9 -> 347.2 mm, vias 8 -> 6
- net /ROW1: vias 12 -> 10
- net /ROW2: vias 7 -> 5
- net GND: vias 41 -> 44

Commit message: sm improvements on pcb, added stabalizers' 3d model and using 2.75u of right space bar instead of 3u
Parts:
- S1: footprint PCM_marbastlib-mx:STAB_MX_3u -> PCM_marbastlib-mx:STAB_MX_2.75u
- moved D60 2.55 mm to (265.6, 198.2)
- moved RGB60 2.33 mm to (256.7, 201.5)
- moved S1 2.33 mm to (255.5, 197.0)
- moved SW60 2.33 mm to (255.5, 197.0)
Routing:
- net /COL4: track 334.1 -> 329.4 mm
- net +5V: track 2380.1 -> 2377.6 mm
- net Net-(RGB59-DOUT): track 34.6 -> 32.1 mm
- net Net-(RGB60-DOUT): track 84.8 -> 87.3 mm
- net /COL9: track 200.9 -> 202.3 mm
- net Net-(RGB54-DOUT): track 331.3 -> 332.4 mm, vias 4 -> 6
- net /ROW4: vias 10 -> 8
- net GND: vias 44 -> 46
- net (no net): vias 0 -> 1
